File: Hardware/JabChip.kicad_pcb (KiCad board)
At the start: 4 copper layers, 25.4 x 25.5 mm, 43 parts, among them J1 USB_C, J2 JSTPH, J4 Piezo-, SW2 434133025816, U1 AP2112K-3.3, U2 MCP73831-2-OT, U3 LSM6DS3, U4 ESP32-S3-WROOM-1

Commit message: fix: Reassign piezo from IO3 to IO9 to avoid JTAG debug
Parts:
- D4: value LED -> LED_R
- D7: value LED -> LED_G
- renumbered P+ to J3, BOOT to SW1
Connections:
- C3 pad 1: +5V -> GND
- C3 pad 2: GND -> +5V
- U4 pad 15: Piezo -> /3
- U4 pad 17: /9 -> Piezo
Routing:
- net Piezo: track 2.47 -> 4.70 mm
Changed lines of the file:
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@@
 	(net 58 "/5")
 	(net 59 "/6")
-	(net 60 "/9")
+	(net 60 "/3")
 	(net 61 "/10")
 	(net 62 "/4")
@@
 			)
 		)
-		(property "Value" "LED"
+		(property "Value" "LED_R"
 			(at 0 1.65 90)
 			(layer "F.Fab")
@@
 			)
 		)
-		(property "Value" "LED"
+		(property "Value" "LED_G"
 			(at 0 1.65 90)
 			(layer "F.Fab")
@@
 		(descr "https://katalog.we-online.com/em/datasheet/434133025816.pdf")
 		(tags "tactile switch Wurth Wuerth")
-		(property "Reference" "BOOT"
+		(property "Reference" "SW1"
 			(at 0 2.7514 0)
 			(layer "F.SilkS")
@@
 		(descr "Wire Pad, Square, SMD Pad,  1mm x 2mm,")
 		(tags "MesurementPoint Square SMDPad 1mmx2mm ")
-		(property "Reference" "P+"
+		(property "Reference" "J3"
 			(at -1.704 0.1016 0)
 			(layer "F.SilkS")
@@
 			(layers "F.Cu" "F.Mask" "F.Paste")
 			(roundrect_rratio 0.25)
-			(net 1 "+5V")
+			(net 2 "GND")
 			(pintype "passive")
 		)
@@
 			(layers "F.Cu" "F.Mask" "F.Paste")
 			(roundrect_rratio 0.25)
-			(net 2 "GND")
+			(net 1 "+5V")
 			(pintype "passive")
 		)
@@
 			(size 1.5 0.9)
 			(layers "B.Cu" "B.Mask" "B.Paste")
-			(net 7 "Piezo")
+			(net 60 "/3")
 			(pinfunction "IO3")
 			(pintype "bidirectional")
@@
 			(size 1.5 0.9)
 			(layers "B.Cu" "B.Mask" "B.Paste")
-			(net 60 "/9")
+			(net 7 "Piezo")
 			(pinfunction "IO9")
 			(pintype "bidirectional")
@@
 	)
 	(segment
-		(start 145.6182 80.4196)
-		(end 145.6182 81.9658)
+		(start 143.0782 80.4196)
+		(end 143.0782 81.3696)
+		(width 0.3)
+		(layer "B.Cu")
+		(net 7)
+	)
+	(segment
+		(start 143.6998 81.9912)
+		(end 145.6436 81.9912)
+		(width 0.3)
+		(layer "B.Cu")
+		(net 7)
+	)
+	(segment
+		(start 143.0782 81.3696)
+		(end 143.6998 81.9912)
 		(width 0.3)
 		(layer "B.Cu")
