File: Hardware/JabChip.kicad_pcb (KiCad board)
At the start: 4 copper layers, 25.4 x 25.5 mm, 43 parts, among them J1 USB_C, J2 JSTPH, J3 Piezo+, J4 Piezo-, SW1 434133025816, SW2 434133025816, U1 AP2112K-3.3, U2 MCP73831-2-OT, U3 LSM6DS3, U4 ESP32-S3-WROOM-1

Commit message: fix: Silkscreen labels
Parts:
- renumbered SW1 to BOOT
Changed lines of the file:
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@@
 			(at 0.15 -2.6 0)
 			(layer "F.SilkS")
+			(hide yes)
 			(effects
 				(font
@@
 		(descr "https://katalog.we-online.com/em/datasheet/434133025816.pdf")
 		(tags "tactile switch Wurth Wuerth")
-		(property "Reference" "SW1"
+		(property "Reference" "BOOT"
 			(at 0 2.7514 0)
 			(layer "F.SilkS")

Commit message: !fix: Correct ESD protection diodes and regenerate gerber output files
Parts:
- turned D2 to 180 degrees
- turned D5 to 0 degrees
- turned D6 to 180 degrees
- renumbered BOOT to SW1
Connections:
- D2 pad 1: GND -> VBUS
- D2 pad 2: VBUS -> GND
- D5 pad 1: GND -> D-
- D5 pad 2: D- -> GND
- D6 pad 1: GND -> D+
- D6 pad 2: D+ -> GND
